File: kicad/80bus.kicad_pcb (KiCad board)
At the start: 2 copper layers, 100 x 203.2 mm, 14 parts, among them J1 Conn_01x80, J2 Conn_01x80, J3 Conn_01x80, J4 Conn_01x80, J5 Conn_01x80, SW1 Reset, T1 Terminal_01x05

Commit message: Kicad 9 and docs
Parts:
- removed H1, H2, H3, H4: MountingHole_3.2mm_M3, MountingHole:MountingHole_3.2mm_M3
- added G001: LOGO, 80bus:qr code, B.Cu at (199.6, 236.2)
Other:
- board text added: "947b8645-6249-4713-a135-48ebccf20ca7"
- board text added: "CS-015"
- board text added: "Documentation -->"
- board text added: "Nascom / Gemini / 80-BUS 5 Slot Backplane Version 2.1"
- board text removed: "Nascom / Gemini / 80-BUS 5 Slot Backplane Version 2.0.1"
- board text removed: "_BAO_"
- board text removed: "c4768bbb-909c-46de-929c-a8bccd0ab267"
