File: kicad/80bus.kicad_sch (KiCad schematic)
At the start: 9 parts, among them J1 Conn_01x80, J2 Conn_01x80, J3 Conn_01x80, J4 Conn_01x80, J5 Conn_01x80, SW1 Reset, T1 Terminal_01x05

Commit message: Kicad 9 and docs
Other:
- title: 80-Bus Card Backplane -> 80-Bus Card Backplane - Kicad 9
